File: boiler_thermostat.kicad_pcb (KiCad board)
At the start: 2 copper layers, 99.1 x 99.1 mm, 9 parts, among them J1 AC_input, J2 Relay_Control, J3 Thermometer, J4 uC, U2 ESP32-WROVER-E

Commit message: dev
Parts:
- J4: value uC -> Control_panel
- moved R1 0.28 mm to (116.8, 121.9)
Connections:
- net /GND renamed /5V-

Commit message: dev
Parts:
- moved R1 3.81 mm to (116.8, 118.1)
- moved J1 2.54 mm to (108.0, 82.5)
- moved J3 2.54 mm to (109.2, 118.1)
- moved PS1 2.54 mm to (121.3, 62.3)
- moved J4 2.54 mm to (113.0, 99.3)
- moved REL1 1.00 mm to (152.9, 85.1)
Changed lines of the file:
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@@
     )
     (pad_to_mask_clearance 0)
+    (aux_axis_origin 104.14 53.34)
+    (grid_origin 104.14 53.34)
     (pcbplotparams
       (layerselection 0x00010fc_ffffffff)
@@
   )
   (footprint "Custom_Terminalblock:Ninigi AC141R-02P-2.54" (layer "F.Cu")
-    (at 107.991 85.09 -90)
+    (at 107.991 82.55 -90)
     (property "Sheetfile" "File: boiler_thermostat.kicad_sch")
     (property "Sheetname" "")
@@
   )
   (footprint "Custom_Connector:RJ45_Keystone_942" (layer "F.Cu")
-    (at 113.03 101.7905 -90)
+    (at 113.03 99.2505 -90)
     (descr "8 Pol Shallow Latch Connector, Modjack, RJ45 (https://cdn.amphenol-icc.com/media/wysiwyg/files/drawing/c-bmj-0102.pdf)")
     (tags "RJ45")
@@
   )
   (footprint "Resistor_SMD:R_1206_3216Metric_Pad1.30x1.75mm_HandSolder" (layer "F.Cu")
-    (at 116.84 121.92 90)
+    (at 116.84 118.11 90)
     (descr "Resistor SMD 1206 (3216 Metric), square (rectangular) end terminal, IPC_7351 nominal with elongated pad for handsoldering. (Body size source: IPC-SM-782 page 72, https://www.pcb-3d.com/wordpress/wp-content/uploads/ipc-sm-782a_amendment_1_and_2.pdf), generated with kicad-footprint-generator")
     (tags "resistor handsolder")
@@
   )
   (footprint "Converter_ACDC:Converter_ACDC_HiLink_HLK-PMxx" (layer "F.Cu")
-    (at 123.8675 62.27)
+    (at 121.3275 62.27)
     (descr "ACDC-Converter, 3W, HiLink, HLK-PMxx, THT, http://www.hlktech.net/product_detail.php?ProId=54")
     (tags "ACDC-Converter 3W THT HiLink board mount module")
@@
   )
   (footprint "TerminalBlock:TerminalBlock_bornier-3_P5.08mm" (layer "F.Cu")
-    (at 109.22 120.65 -90)
+    (at 109.22 118.11 -90)
     (descr "simple 3-pin terminal block, pitch 5.08mm, revamped version of bornier3")
     (tags "terminal block bornier3")
@@
     (property "ki_keywords" "connector")
     (attr through_hole)
-    (fp_text reference "J3" (at 8.89 -7.62 90) (layer "F.SilkS")
+    (fp_text reference "J3" (at 11.43 -7.62 90) (layer "F.SilkS")
         (effects (font (size 3 3) (thickness 0.5)))
     )
@@
   )
   (footprint "Custom_Relay:RELC-2CH-5V-UNI" (layer "F.Cu")
-    (at 153.67 84.455)
+    (at 152.908 85.099026)
     (fp_text reference "REL1" (at 22.86 41.275 unlocked) (layer "F.SilkS")
         (effects (font (size 3 3) (thickness 0.5)))
@@
     (fp_arc (start 47.244 35.687) (mid 46.44952 37.388796) (end 44.704 38.081949)
       (stroke (width 0.12) (type default)) (layer "F.SilkS"))
-    (fp_circle (center 0 0) (end 1.550233 0)
+    (fp_circle (center 0 0) (end 1.6 0)
       (stroke (width 0.12) (type default)) (fill none) (layer "Edge.Cuts"))
-    (fp_circle (center 0 35.56) (end 1.550233 35.56)
+    (fp_circle (center 0 35.56) (end 1.6 35.56)
       (stroke (width 0.12) (type default)) (fill none) (layer "Edge.Cuts"))
-    (fp_circle (center 44.704 0) (end 46.254233 0)
+    (fp_circle (center 44.704 0) (end 46.304 0)
       (stroke (width 0.12) (type default)) (fill none) (layer "Edge.Cuts"))
-    (fp_circle (center 44.704 35.56) (end 46.254233 35.56)
+    (fp_circle (center 44.704 35.56) (end 46.304 35.56)
       (stroke (width 0.12) (type default)) (fill none) (layer "Edge.Cuts"))
   )

Commit message: dev
Connections:
- J2 pad 1: Net-(J2-Pin_1) -> /5V+
- J2 pad 2: /5V- -> /GND
- J3 pad 3: /5V- -> /GND
- J4 pad 1: Net-(J2-Pin_1) -> /GND
- J4 pad 2: /3V3+ -> /5V+
- J4 pad 3: /5V- -> /3V3+
- J4 pad 4: unconnected-(J4-Pad4) -> /I2C_SDA
- J4 pad 5: unconnected-(J4-Pad5) -> /I2C_SCL
- J4 pad 8: unconnected-(J4-Pad8) -> /BTN1
- PS1 pad 3: /5V- -> /GND
- PS1 pad 4: Net-(J2-Pin_1) -> /5V+
- U1 pad 1: Net-(J2-Pin_1) -> /5V+
- U1 pad 2: /5V- -> /GND
- U1 pad 4: /5V- -> /GND
- U2 pad 1: /5V- -> /GND
- U2 pad 15: /5V- -> /GND
- U2 pad 23: unconnected-(U2-IO15) -> Net-(J3-Pin_2)
- U2 pad 31: unconnected-(U2-IO19) -> /BTN1
- U2 pad 33: unconnected-(U2-IO21) -> /I2C_SDA
- U2 pad 36: unconnected-(U2-IO22) -> /I2C_SCL
- U2 pad 38: /5V- -> /GND

Commit message: dev
Connections:
- J4 pad 6: unconnected-(J4-Pad6) -> /BTN_UP
- J4 pad 7: unconnected-(J4-Pad7) -> /BTN_DOWN
- J4 pad 8: /BTN1 -> unconnected-(J4-Pad8)
- U2 pad 16: unconnected-(U2-IO13) -> Net-(J2-Pin_3)
- U2 pad 30: unconnected-(U2-IO18) -> /BTN_DOWN
- U2 pad 31: /BTN1 -> /BTN_UP
Routing:
- net /3V3+: track 0.00 -> 177.5 mm
- net /5V+: track 0.00 -> 108.4 mm
- net Net-(J2-Pin_3): track 0.00 -> 101.8 mm
- net /I2C_SDA: track 0.00 -> 48.7 mm, vias 0 -> 1
- net /I2C_SCL: track 0.00 -> 48.2 mm, vias 0 -> 1
- net /BTN_UP: track 0.00 -> 40.8 mm, vias 0 -> 1
- net /BTN_DOWN: track 0.00 -> 37.2 mm, vias 0 -> 1
- net Net-(J3-Pin_2): track 0.00 -> 20.1 mm
- added copper zone on B.Cu, net /AC_LINE
- added copper zone on F.Cu, net /AC_LINE
- added copper zone on B.Cu, net /AC_NULL
- added copper zone on F.Cu, net /AC_NULL
- added copper zone on B.Cu, net /GND
- added copper zone on F.Cu, net /GND
