File: boiler_thermostat.kicad_sch (KiCad schematic)
At the start: 8 parts, among them J1 AC_input, J2 Relay_Control, J3 Thermometer, J4 uC, U2 ESP32-WROVER-E

Commit message: dev
Parts:
- J4: value uC -> Control_panel
Changed lines of the file:
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@@
     (pin "2")
     (instances
-      (project "Boiler_termostat"
+      (project "boiler_thermostat"
         (path "/7f07eb40-58fa-446e-a670-e70b13e07761"
           (reference "J1") (unit 1) (value "AC_input") (footprint "Custom_Terminalblock:Ninigi AC141R-02P-2.54")
@@
     (pin "4")
     (instances
-      (project "Boiler_termostat"
+      (project "boiler_thermostat"
         (path "/7f07eb40-58fa-446e-a670-e70b13e07761"
           (reference "U1") (unit 1) (value "~") (footprint "Custom_Converter:DCDC_Mini560")
@@
       (effects (font (size 1.27 1.27)) (justify right))
     )
-    (property "Value" "uC" (at 205.74 48.895 0)
+    (property "Value" "Control_panel" (at 205.74 48.895 0)
       (effects (font (size 1.27 1.27)) (justify right))
     )
@@
     (pin "8")
     (instances
-      (project "Boiler_termostat"
-        (path "/7f07eb40-58fa-446e-a670-e70b13e07761"
-          (reference "J4") (unit 1) (value "uC") (footprint "Custom_Connector:RJ45_Keystone_942")
+      (project "boiler_thermostat"
+        (path "/7f07eb40-58fa-446e-a670-e70b13e07761"
+          (reference "J4") (unit 1) (value "Control_panel") (footprint "Custom_Connector:RJ45_Keystone_942")
         )
       )
@@
     (pin "4")
     (instances
-      (project "Boiler_termostat"
+      (project "boiler_thermostat"
         (path "/7f07eb40-58fa-446e-a670-e70b13e07761"
           (reference "J2") (unit 1) (value "Relay_Control") (footprint "TerminalBlock:TerminalBlock_bornier-4_P5.08mm")
@@
     (pin "3")
     (instances
-      (project "Boiler_termostat"
+      (project "boiler_thermostat"
         (path "/7f07eb40-58fa-446e-a670-e70b13e07761"
           (reference "J3") (unit 1) (value "Thermometer") (footprint "TerminalBlock:TerminalBlock_bornier-3_P5.08mm")
@@
     (pin "4")
     (instances
-      (project "Boiler_termostat"
+      (project "boiler_thermostat"
         (path "/7f07eb40-58fa-446e-a670-e70b13e07761"
           (reference "PS1") (unit 1) (value "HLK-PM01") (footprint "Converter_ACDC:Converter_ACDC_HiLink_HLK-PMxx")
@@
     (pin "2")
     (instances
-      (project "Boiler_termostat"
+      (project "boiler_thermostat"
         (path "/7f07eb40-58fa-446e-a670-e70b13e07761"
           (reference "R1") (unit 1) (value "R") (footprint "Resistor_SMD:R_1206_3216Metric_Pad1.30x1.75mm_HandSolder")
@@
     (pin "9")
     (instances
-      (project "Boiler_termostat"
+      (project "boiler_thermostat"
         (path "/7f07eb40-58fa-446e-a670-e70b13e07761"
           (reference "U2") (unit 1) (value "ESP32-WROVER-E") (footprint "Custom_RF_Module:ESP32-WROVER-IE")

Commit message: dev
Connections:
- net 3V3+: now also J4.3; no longer J4.2
- net 5V+: now reaches J2.1 (Pin_1), PS1.4 (+Vout), U1.1 (IN+)
- net 5V+: now also J4.2; no longer J4.1
- net I2C_SDA: now reaches J4.4
- net I2C_SDA: now also U2.33 (IO21)
- net I2C_SCL: now reaches J4.5
- net I2C_SCL: now also U2.36 (IO22)
- net BTN1: now reaches J4.8
- net BTN1: now also U2.31 (IO19)
- net at J3.2 (Pin_2), R1.1: now also U2.23 (IO15)
- net 5V- renamed GND
- net GND: now also J4.1; no longer J4.3
Changed lines of the file:
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@@
   (junction (at 158.75 73.66) (diameter 0) (color 0 0 0 0)
   )
+  (junction (at 170.18 55.88) (diameter 0) (color 0 0 0 0)
+  )
   (junction (at 140.97 99.06) (diameter 0) (color 0 0 0 0)
   )
@@
     (stroke (width 0) (type default))
   )
-  (wire (pts (xy 186.69 36.83) (xy 186.69 38.1))
-    (stroke (width 0) (type default))
-  )
   (wire (pts (xy 185.42 99.06) (xy 185.42 91.44))
     (stroke (width 0) (type default))
   )
-  (wire (pts (xy 186.69 43.18) (xy 179.07 43.18))
+  (wire (pts (xy 181.61 48.26) (xy 186.69 48.26))
+    (stroke (width 0) (type default))
+  )
+  (wire (pts (xy 191.77 69.85) (xy 173.99 69.85))
     (stroke (width 0) (type default))
   )
@@
     (stroke (width 0) (type default))
   )
+  (wire (pts (xy 181.61 49.53) (xy 181.61 48.26))
+    (stroke (width 0) (type default))
+  )
+  (wire (pts (xy 189.23 71.12) (xy 189.23 137.16))
+    (stroke (width 0) (type default))
+  )
+  (wire (pts (xy 177.8 36.83) (xy 177.8 40.64))
+    (stroke (width 0) (type default))
+  )
   (wire (pts (xy 144.78 101.6) (xy 138.43 101.6))
     (stroke (width 0) (type default))
   )
+  (wire (pts (xy 194.31 116.84) (xy 185.42 116.84))
+    (stroke (width 0) (type default))
+  )
   (wire (pts (xy 179.07 46.99) (xy 172.72 46.99))
     (stroke (width 0) (type default))
@@
     (stroke (width 0) (type default))
   )
+  (wire (pts (xy 185.42 111.76) (xy 191.77 111.76))
+    (stroke (width 0) (type default))
+  )
   (wire (pts (xy 135.89 53.34) (xy 135.89 36.83))
     (stroke (width 0) (type default))
@@
     (stroke (width 0) (type default))
   )
-  (wire (pts (xy 186.69 40.64) (xy 177.8 40.64))
-    (stroke (width 0) (type default))
-  )
   (wire (pts (xy 172.72 91.44) (xy 185.42 91.44))
     (stroke (width 0) (type default))
@@
     (stroke (width 0) (type default))
   )
+  (wire (pts (xy 186.69 55.88) (xy 186.69 67.31))
+    (stroke (width 0) (type default))
+  )
   (wire (pts (xy 158.75 78.74) (xy 158.75 73.66))
     (stroke (width 0) (type default))
   )
+  (wire (pts (xy 173.99 48.26) (xy 180.34 48.26))
+    (stroke (width 0) (type default))
+  )
   (wire (pts (xy 138.43 78.74) (xy 158.75 78.74))
     (stroke (width 0) (type default))
@@
     (stroke (width 0) (type default))
   )
+  (wire (pts (xy 194.31 67.31) (xy 194.31 116.84))
+    (stroke (width 0) (type default))
+  )
+  (wire (pts (xy 185.42 104.14) (xy 193.04 104.14))
+    (stroke (width 0) (type default))
+  )
   (wire (pts (xy 172.72 44.45) (xy 172.72 46.99))
     (stroke (width 0) (type default))
   )
-  (wire (pts (xy 135.89 36.83) (xy 186.69 36.83))
+  (wire (pts (xy 180.34 48.26) (xy 180.34 45.72))
+    (stroke (width 0) (type default))
+  )
+  (wire (pts (xy 189.23 137.16) (xy 185.42 137.16))
     (stroke (width 0) (type default))
   )
@@
     (stroke (width 0) (type default))
   )
+  (wire (pts (xy 170.18 71.12) (xy 189.23 71.12))
+    (stroke (width 0) (type default))
+  )
   (wire (pts (xy 113.03 83.82) (xy 113.03 86.36))
     (stroke (width 0) (type default))
   )
+  (wire (pts (xy 179.07 38.1) (xy 179.07 46.99))
+    (stroke (width 0) (type default))
+  )
+  (wire (pts (xy 173.99 69.85) (xy 173.99 48.26))
+    (stroke (width 0) (type default))
+  )
   (wire (pts (xy 161.29 45.72) (xy 162.56 45.72))
     (stroke (width 0) (type default))
@@
     (stroke (width 0) (type default))
   )
-  (wire (pts (xy 179.07 43.18) (xy 179.07 46.99))
+  (wire (pts (xy 186.69 67.31) (xy 194.31 67.31))
     (stroke (width 0) (type default))
   )
@@
     (stroke (width 0) (type default))
   )
+  (wire (pts (xy 179.07 38.1) (xy 186.69 38.1))
+    (stroke (width 0) (type default))
+  )
   (wire (pts (xy 138.43 73.66) (xy 138.43 78.74))
     (stroke (width 0) (type default))
   )
+  (wire (pts (xy 193.04 104.14) (xy 193.04 68.58))
+    (stroke (width 0) (type default))
+  )
+  (wire (pts (xy 170.18 55.88) (xy 170.18 71.12))
+    (stroke (width 0) (type default))
+  )
   (wire (pts (xy 127 69.85) (xy 135.89 69.85))
     (stroke (width 0) (type default))
   )
+  (wire (pts (xy 191.77 111.76) (xy 191.77 69.85))
+    (stroke (width 0) (type default))
+  )
   (wire (pts (xy 144.78 134.62) (xy 140.97 134.62))
     (stroke (width 0) (type default))
@@
     (stroke (width 0) (type default))
   )
-  (wire (pts (xy 177.8 40.64) (xy 177.8 45.72))
+  (wire (pts (xy 193.04 68.58) (xy 175.26 68.58))
+    (stroke (width 0) (type default))
+  )
+  (wire (pts (xy 180.34 45.72) (xy 186.69 45.72))
     (stroke (width 0) (type default))
   )
@@
     (stroke (width 0) (type default))
   )
+  (wire (pts (xy 177.8 45.72) (xy 177.8 43.18))
+    (stroke (width 0) (type default))
+  )
   (wire (pts (xy 95.25 53.34) (xy 111.76 53.34))
     (stroke (width 0) (type default))
   )
+  (wire (pts (xy 175.26 49.53) (xy 175.26 68.58))
+    (stroke (width 0) (type default))
+  )
+  (wire (pts (xy 177.8 43.18) (xy 186.69 43.18))
+    (stroke (width 0) (type default))
+  )
   (wire (pts (xy 138.43 101.6) (xy 138.43 90.17))
     (stroke (width 0) (type default))
   )
+  (wire (pts (xy 177.8 40.64) (xy 186.69 40.64))
+    (stroke (width 0) (type default))
+  )
   (wire (pts (xy 113.03 81.28) (xy 132.08 81.28))
     (stroke (width 0) (type default))
   )
+  (wire (pts (xy 135.89 36.83) (xy 177.8 36.83))
+    (stroke (width 0) (type default))
+  )
+  (wire (pts (xy 175.26 49.53) (xy 181.61 49.53))
+    (stroke (width 0) (type default))
+  )
   (wire (pts (xy 140.97 134.62) (xy 140.97 99.06))
     (stroke (width 0) (type default))
@@
     (effects (font (size 1.27 1.27)) (justify left bottom))
   )
+  (label "I2C_SCL" (at 185.42 104.14 0) (fields_autoplaced)
+    (effects (font (size 1.27 1.27)) (justify left bottom))
+  )
   (label "3V3+" (at 158.75 69.85 0) (fields_autoplaced)
     (effects (font (size 1.27 1.27)) (justify left bottom))
@@
     (effects (font (size 1.27 1.27)) (justify left bottom))
   )
-  (label "5V-" (at 132.08 58.42 0) (fields_autoplaced)
-    (effects (font (size 1.27 1.27)) (justify left bottom))
-  )
+  (label "BTN1" (at 185.42 116.84 0) (fields_autoplaced)
+    (effects (font (size 1.27 1.27)) (justify left bottom))
+  )
+  (label "I2C_SDA" (at 185.42 111.76 0) (fields_autoplaced)
+    (effects (font (size 1.27 1.27)) (justify left bottom))
+  )
+  (label "5V+" (at 132.08 53.34 0) (fields_autoplaced)
+    (effects (font (size 1.27 1.27)) (justify left bottom))
+  )

Commit message: dev
Connections:
- net BTN_UP: now reaches J4.6
- net BTN_UP: now also U2.31 (IO19)
- net BTN_DOWN: now reaches J4.7
- net BTN_DOWN: now also U2.30 (IO18)
- net at J2.3 (Pin_3), J2.4 (Pin_4): now also U2.16 (IO13)
- net BTN1: no longer names the net of J4.8
- net BTN1: no longer U2.31 (IO19)
Changed lines of the file:
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@@
 (kicad_sch (version 20221004) (generator eeschema)
   (paper "A4")
+  (junction (at 113.03 86.36) (diameter 0) (color 0 0 0 0)
+  )
   (junction (at 162.56 45.72) (diameter 0) (color 0 0 0 0)
   )
@@
     (stroke (width 0) (type default))
   )
+  (wire (pts (xy 113.03 86.36) (xy 113.03 137.16))
+    (stroke (width 0) (type default))
+  )
   (wire (pts (xy 177.8 36.83) (xy 177.8 40.64))
     (stroke (width 0) (type default))
@@
     (stroke (width 0) (type default))
   )
+  (wire (pts (xy 185.42 119.38) (xy 195.58 119.38))
+    (stroke (width 0) (type default))
+  )
   (wire (pts (xy 161.29 69.85) (xy 161.29 90.17))
     (stroke (width 0) (type default))
@@
     (stroke (width 0) (type default))
   )
+  (wire (pts (xy 176.53 50.8) (xy 186.69 50.8))
+    (stroke (width 0) (type default))
+  )
   (wire (pts (xy 162.56 45.72) (xy 162.56 55.88))
     (stroke (width 0) (type default))
@@
     (stroke (width 0) (type default))
   )
-  (wire (pts (xy 186.69 55.88) (xy 186.69 67.31))
-    (stroke (width 0) (type default))
-  )
   (wire (pts (xy 158.75 78.74) (xy 158.75 73.66))
     (stroke (width 0) (type default))
@@
     (stroke (width 0) (type default))
   )
+  (wire (pts (xy 176.53 67.31) (xy 176.53 50.8))
+    (stroke (width 0) (type default))
+  )
   (wire (pts (xy 138.43 78.74) (xy 158.75 78.74))
     (stroke (width 0) (type default))
@@
     (stroke (width 0) (type default))
   )
+  (wire (pts (xy 177.8 53.34) (xy 186.69 53.34))
+    (stroke (width 0) (type default))
+  )
   (wire (pts (xy 185.42 104.14) (xy 193.04 104.14))
     (stroke (width 0) (type default))
@@
     (stroke (width 0) (type default))
   )
+  (wire (pts (xy 177.8 66.04) (xy 177.8 53.34))
+    (stroke (width 0) (type default))
+  )
   (wire (pts (xy 180.34 48.26) (xy 180.34 45.72))
     (stroke (width 0) (type default))
@@
     (stroke (width 0) (type default))
   )
+  (wire (pts (xy 195.58 66.04) (xy 177.8 66.04))
+    (stroke (width 0) (type default))
+  )
   (wire (pts (xy 127 78.74) (xy 127 69.85))
     (stroke (width 0) (type default))
@@
     (stroke (width 0) (type default))
   )
-  (wire (pts (xy 186.69 67.31) (xy 194.31 67.31))
+  (wire (pts (xy 176.53 67.31) (xy 194.31 67.31))
     (stroke (width 0) (type default))
   )
@@
     (stroke (width 0) (type default))
   )
+  (wire (pts (xy 195.58 119.38) (xy 195.58 66.04))
+    (stroke (width 0) (type default))
+  )
   (wire (pts (xy 191.77 111.76) (xy 191.77 69.85))
     (stroke (width 0) (type default))
@@
     (stroke (width 0) (type default))
   )
+  (wire (pts (xy 113.03 137.16) (xy 144.78 137.16))
+    (stroke (width 0) (type default))
+  )
   (wire (pts (xy 95.25 53.34) (xy 111.76 53.34))
     (stroke (width 0) (type default))
@@
     (effects (font (size 1.27 1.27)) (justify left bottom))
   )
-  (label "BTN1" (at 185.42 116.84 0) (fields_autoplaced)
+  (label "BTN_UP" (at 185.42 116.84 0) (fields_autoplaced)
+    (effects (font (size 1.27 1.27)) (justify left bottom))
+  )
+  (label "BTN_DOWN" (at 185.42 119.38 0) (fields_autoplaced)
     (effects (font (size 1.27 1.27)) (justify left bottom))
   )
@@
     (effects (font (size 1.27 1.27)) (justify left bottom))
   )
+  (netclass_flag "" (length 2.54) (shape round) (at 105.41 57.15 0) (fields_autoplaced)
+    (effects (font (size 1.27 1.27)) (justify left bottom))
+    (property "Netclass" "AC" (at 106.1085 54.61 0)
+      (effects (font (size 1.27 1.27) italic) (justify left))
+    )
+  )
+  (netclass_flag "" (length 2.54) (shape round) (at 105.41 53.34 0) (fields_autoplaced)
+    (effects (font (size 1.27 1.27)) (justify left bottom))
+    (property "Netclass" "AC" (at 106.1085 50.8 0)
+      (effects (font (size 1.27 1.27) italic) (justify left))
+    )
+  )
   (symbol (lib_id "Connector_Generic:Conn_01x02") (at 90.17 54.61 0) (mirror y) (unit 1)
